File: ColumnDriver.kicad_sch (KiCad schematic)
At the start: 112 parts, among them Q10 AP4606, Q11 AP4606, Q12 AP4606, Q13 AP4606, Q14 AP4606, Q15 AP4606, Q16 AP4606, Q17 AP4606, Q18 AP4606, Q19 AP4606, Q20 AP4606, Q21 AP4606, Q22 AP4606, Q23 AP4606, Q24 AP4606, Q25 AP4606, Q26 AP4606, Q27 AP4606, Q28 AP4606, Q29 AP4606, Q3 AP4606, Q30 AP4606, Q4 AP4606, Q5 AP4606, Q6 AP4606, Q7 AP4606, Q8 AP4606, Q9 AP4606

Commit message: Add subrevision, reference submodule objects
Parts:
- Q10, Q11, Q12, Q13, Q14, Q15, Q16, Q17, Q18, Q19, Q20, Q21, Q22, Q23, Q24, Q25, Q26, Q27, Q28, Q29, Q3, Q30, Q4, Q5, Q6, Q7, Q8, Q9: footprint Package_SO:SOIC-8_3.9x4.9mm_P1.27mm -> Package_SO:SOP-8_3.9x4.9mm_P1.27mm; symbol FlippyDriver:DMC3021LSD -> Nieto_Driver_FET:AP4606

Commit message: Initial draft of Revision D
- Remove I2C Bus, and replace with PWM Input
- Remove temp sensors due to no I2C bus
- Add 5V aux output from 24V, supports LM7805 (w/ Heatsink) and VX7805
- Larger components for high current nets
Parts:
- Q10, Q11, Q12, Q13, Q14, Q15, Q16, Q17, Q18, Q19, Q20, Q21, Q22, Q23, Q24, Q25, Q26, Q27, Q28, Q29, Q3, Q30, Q4, Q5, Q6, Q7, Q8, Q9: footprint Package_SO:SOP-8_3.9x4.9mm_P1.27mm -> Package_SO:SOIC-8_3.9x4.9mm_P1.27mm
