File: RowDriver.kicad_sch (KiCad schematic)
At the start: 64 parts, among them Q31 AP4606, Q32 AP4606, Q33 AP4606, Q34 AP4606, Q35 AP4606, Q36 AP4606, Q37 AP4606, Q38 AP4606, Q39 AP4606, Q40 AP4606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

Commit message: Add subrevision, reference submodule objects
Parts:
- Q31, Q32, Q33, Q34, Q35, Q36, Q37, Q38, Q39, Q40, Q41, Q42, Q43, Q44, Q45, Q46: footprint Package_SO:SOIC-8_3.9x4.9mm_P1.27mm -> Package_SO:SOP-8_3.9x4.9mm_P1.27mm; symbol FlippyDriver:DMC3021LSD -> Nieto_Driver_FET:AP4606

Commit message: Add images and 3D models
Parts:
- Q31, Q32, Q33, Q34, Q35, Q36, Q37, Q38, Q39, Q40, Q41, Q42, Q43, Q44, Q45, Q46: footprint Package_SO:SOP-8_3.9x4.9mm_P1.27mm -> Package_SO:SOIC-8_3.9x4.9mm_P1.27mm
